File: hardware/servodriver.brd (EAGLE design)
At the start: 76.2 x 50.8 mm, 21 parts, among them IC1 PIC12F683P, IC2 7805

Commit message: Add the CAM files
Other:
- board text added: "ServoDriver 2014-04-05 Stockton Marine Science Program"
- board text removed: "ServoDriver 2014-04-04 Stockton Marine Science Program"
Changed lines of the file:
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@@
 <wire x1="76.2" y1="50.8" x2="0" y2="50.8" width="0" layer="20"/>
 <wire x1="0" y1="50.8" x2="0" y2="0" width="0" layer="20"/>
-<text x="2.54" y="40.005" size="1.778" layer="46" rot="R270">-  +</text>
-<text x="14.605" y="41.91" size="1.778" layer="46">ServoDriver 2014-04-04
+<text x="1.905" y="40.005" size="1.778" layer="46" rot="R270">-  +</text>
+<text x="14.605" y="41.91" size="1.778" layer="46">ServoDriver 2014-04-05
 Stockton Marine Science Program</text>
-<text x="3.81" y="40.005" size="1.778" layer="46" rot="MR270">-  +</text>
 <text x="13.97" y="1.27" size="1.778" layer="46">B R Y</text>
 <text x="3.81" y="27.305" size="1.778" layer="46">7-12V DC</text>

Commit message: Update hardware details, including a BOM
Parts:
- R3, R4: value 150R -> 620R
Changed lines of the file:
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@@
 </element>
 <element name="LED1" library="led" package="LED3MM" value="" x="20.32" y="29.21" rot="R180"/>
-<element name="R3" library="rcl" package="0207/10" value="150R" x="33.02" y="29.21"/>
+<element name="R3" library="rcl" package="0207/10" value="620R" x="33.02" y="29.21"/>
 <element name="LED2" library="led" package="LED3MM" value="" x="20.32" y="22.86" rot="R180"/>
-<element name="R4" library="rcl" package="0207/10" value="150R" x="27.94" y="26.035"/>
+<element name="R4" library="rcl" package="0207/10" value="620R" x="27.94" y="26.035"/>
 </elements>
 <signals>
